Commit message: 璇玑工业机器人训练测试生效.

File: legged_lab/assets/xuanji/rb160w/urdf/RB160W.urdf (robot description, URDF)
Before this commit: robot RB160W, 17 links, 16 joints
Links:
- link FL_WHEEL: geometry visual mesh filename=package://RB160W/meshes/FL_WHEEL.STL
- link FL_calf: geometry collision box size=0.05 0.0199999996 0.200000003; visual mesh filename=package://RB160W/meshes/FL_calf.STL
- link FL_hip: geometry visual mesh filename=package://RB160W/meshes/FL_hip.STL
- link FL_thigh: geometry collision box size=0.100000001 0.100000001 0.200000003; visual mesh filename=package://RB160W/meshes/FL_thigh.STL
- link FR_WHEEL: geometry visual mesh filename=package://RB160W/meshes/FR_WHEEL.STL
- link FR_calf: geometry collision box size=0.05 0.02 0.2; visual mesh filename=package://RB160W/meshes/FR_calf.STL
- link FR_hip: geometry visual mesh filename=package://RB160W/meshes/FR_hip.STL
- link FR_thigh: geometry collision box size=0.100000001 0.100000001 0.200000003; visual mesh filename=package://RB160W/meshes/FR_thigh.STL
- link RL_WHEEL: geometry visual mesh filename=package://RB160W/meshes/RL_WHEEL.STL
- link RL_calf: geometry collision box size=0.05 0.0199999996 0.200000003; visual mesh filename=package://RB160W/meshes/RL_calf.STL
- link RL_hip: geometry visual mesh filename=package://RB160W/meshes/RL_hip.STL
- link RL_thigh: geometry collision box size=0.1 0.1 0.2; visual mesh filename=package://RB160W/meshes/RL_thigh.STL
- link RR_WHEEL: geometry visual mesh filename=package://RB160W/meshes/RR_WHEEL.STL
- link RR_calf: geometry collision box size=0.05 0.0199999996 0.200000003; visual mesh filename=package://RB160W/meshes/RR_calf.STL
- link RR_hip: geometry visual mesh filename=package://RB160W/meshes/RR_hip.STL
- link RR_thigh: geometry collision box size=0.100000001 0.100000001 0.200000003; visual mesh filename=package://RB160W/meshes/RR_thigh.STL
- link base_link: geometry collision box size=0.500000007 0.300000004 0.200000003; visual mesh filename=package://RB160W/meshes/base_link.STL
Joints:
- joint FR_WHEEL_joint: axis 0 -1 0 -> 0 1 0
- joint RR_calf_joint: axis 0 -1 0 -> 0 1 0

File: legged_lab/assets/xuanji/rb160w/urdf/RB160W_isaaclab.urdf (robot description, URDF)
Before this commit: robot RB160W, 17 links, 16 joints
Links:
- link FL_WHEEL: geometry visual mesh filename=../meshes/FL_WHEEL.STL
- link FL_calf: geometry collision box size=0.05 0.0199999996 0.200000003; visual mesh filename=../meshes/FL_calf.STL
- link FL_hip: geometry visual mesh filename=../meshes/FL_hip.STL
- link FL_thigh: geometry collision box size=0.100000001 0.100000001 0.200000003; visual mesh filename=../meshes/FL_thigh.STL
- link FR_WHEEL: geometry visual mesh filename=../meshes/FR_WHEEL.STL
- link FR_calf: geometry collision box size=0.05 0.02 0.2; visual mesh filename=../meshes/FR_calf.STL
- link FR_hip: geometry visual mesh filename=../meshes/FR_hip.STL
- link FR_thigh: geometry collision box size=0.100000001 0.100000001 0.200000003; visual mesh filename=../meshes/FR_thigh.STL
- link RL_WHEEL: geometry visual mesh filename=../meshes/RL_WHEEL.STL
- link RL_calf: geometry collision box size=0.05 0.0199999996 0.200000003; visual mesh filename=../meshes/RL_calf.STL
- link RL_hip: geometry visual mesh filename=../meshes/RL_hip.STL
- link RL_thigh: geometry collision box size=0.1 0.1 0.2; visual mesh filename=../meshes/RL_thigh.STL
- link RR_WHEEL: geometry visual mesh filename=../meshes/RR_WHEEL.STL
- link RR_calf: geometry collision box size=0.05 0.0199999996 0.200000003; visual mesh filename=../meshes/RR_calf.STL
- link RR_hip: geometry visual mesh filename=../meshes/RR_hip.STL
- link RR_thigh: geometry collision box size=0.100000001 0.100000001 0.200000003; visual mesh filename=../meshes/RR_thigh.STL
- link base_link: geometry collision box size=0.500000007 0.300000004 0.200000003; visual mesh filename=../meshes/base_link.STL
Joints:
- joint FR_WHEEL_joint: axis 0 -1 0 -> 0 1 0
- joint RR_calf_joint: axis 0 -1 0 -> 0 1 0

File: legged_lab/assets/xuanji/rb160w/urdf/RB160W_isaaclab_actuated.urdf (robot description, URDF)
Before this commit: robot RB160W, 17 links, 16 joints
Links:
- link FL_WHEEL: geometry visual mesh filename=../meshes/FL_WHEEL.STL
- link FL_calf: geometry collision box size=0.05 0.0199999996 0.200000003; visual mesh filename=../meshes/FL_calf.STL
- link FL_hip: geometry visual mesh filename=../meshes/FL_hip.STL
- link FL_thigh: geometry collision box size=0.100000001 0.100000001 0.200000003; visual mesh filename=../meshes/FL_thigh.STL
- link FR_WHEEL: geometry visual mesh filename=../meshes/FR_WHEEL.STL
- link FR_calf: geometry collision box size=0.05 0.02 0.2; visual mesh filename=../meshes/FR_calf.STL
- link FR_hip: geometry visual mesh filename=../meshes/FR_hip.STL
- link FR_thigh: geometry collision box size=0.100000001 0.100000001 0.200000003; visual mesh filename=../meshes/FR_thigh.STL
- link RL_WHEEL: geometry visual mesh filename=../meshes/RL_WHEEL.STL
- link RL_calf: geometry collision box size=0.05 0.0199999996 0.200000003; visual mesh filename=../meshes/RL_calf.STL
- link RL_hip: geometry visual mesh filename=../meshes/RL_hip.STL
- link RL_thigh: geometry collision box size=0.1 0.1 0.2; visual mesh filename=../meshes/RL_thigh.STL
- link RR_WHEEL: geometry visual mesh filename=../meshes/RR_WHEEL.STL
- link RR_calf: geometry collision box size=0.05 0.0199999996 0.200000003; visual mesh filename=../meshes/RR_calf.STL
- link RR_hip: geometry visual mesh filename=../meshes/RR_hip.STL
- link RR_thigh: geometry collision box size=0.100000001 0.100000001 0.200000003; visual mesh filename=../meshes/RR_thigh.STL
- link base_link: geometry collision box size=0.500000007 0.300000004 0.200000003; visual mesh filename=../meshes/base_link.STL
Joints:
- joint FL_thigh_joint: axis 0 -1 0 -> 0 1 0
- joint FR_WHEEL_joint: axis 0 -1 0 -> 0 1 0
- joint RL_thigh_joint: axis 0 -1 0 -> 0 1 0
- joint RR_WHEEL_joint: axis 0 -1 0 -> 0 1 0
- joint RR_calf_joint: axis 0 -1 0 -> 0 1 0
